Commit message: Added gazebo pluggins and fixed inertial issues

File: urdf/camera.xacro (robot description, xacro)
@@ -18,5 +18,5 @@
             </geometry>
         </collision>
-        <box_inertial m="0.2" l="${camera_length}" w="${camera_width}" h="${camera_height}" xyz="0 0 0" rpy="0 0 0" />
+        <xacro:box_inertial m="0.2" l="${camera_length}" w="${camera_width}" h="${camera_height}" xyz="0 0 0" rpy="0 0 0" />
     </link>
     <joint name="base_camera" type="fixed" >
@@ -27,4 +27,12 @@
     <gazebo reference="camera" >
         <material>Gazebo/Black</material>
+        <sensor name="camera_sensor" type="camera">
+            <pose>0 0 0 0 0 0</pose>
+            <visualize>true</visualize>
+            <update_rate>10.0</update_rate>
+            <plugin name="camera_controller" filename="libgazebo_ros_camera.so">
+                <frame_name>camera</frame_name>
+            </plugin>
+        </sensor>
     </gazebo>
 </robot>

File: urdf/robot_arm.xacro (robot description, xacro)
@@ -29,5 +29,5 @@
         <parent link="main_base" />
         <child link="arm_base" />
-        <origin xyz="0 0 ${0.5*(main_base_height+arm_base_height)}" rpy="0 0 0" />
+        <origin xyz="${main_base_length/4} 0 ${0.5*(main_base_height+arm_base_height)}" rpy="0 0 0" />
     </joint>
     <link name="fore_arm">
@@ -43,8 +43,8 @@
                 <cylinder radius="${arm_radius}" length="${arm_length}" />
             </geometry>
-            <origin xyz="0 0 0" rpy="0 0 0" />
+            <origin xyz="0 0 ${0.5*arm_length}" rpy="0 0 0" />
         </collision>
         <xacro:cylinder_inertial m="${arm_mass}" r="${arm_radius}" l="${arm_length}"
-                                     xyz="0 0 0" rpy="0 0 0" />
+                                     xyz="0 0 ${0.5*arm_length}" rpy="0 0 0" />
     </link>
     <joint name="forearm_to_base" type="revolute">
@@ -71,5 +71,5 @@
         </collision>
         <xacro:cylinder_inertial m="${arm_mass}" r="${arm_radius}" l="${arm_length}"
-                                     xyz="0 0 0" rpy="0 0 0" />
+                                     xyz="0 0 ${0.5*arm_length}" rpy="0 0 0" />
     </link>
     <joint name="hand_to_forearm" type="revolute">
@@ -81,3 +81,15 @@
         <limit effort="100" velocity="100" lower="0" upper="${pi/2}" />
     </joint>
+    <gazebo>
+        <plugin name="joint_state_publisher_controller" filename="libgazebo_ros_joint_state_publisher.so">
+            <update_rate>10</update_rate>
+            <joint_name>forearm_to_base</joint_name>
+            <joint_name>hand_to_forearm</joint_name>
+        </plugin>
+    </gazebo>
+    <gazebo>
+        <plugin name="joint_pose_trajectory_controller" filename="libgazebo_ros_joint_pose_trajectory.so">
+            <update_rate>2</update_rate>
+        </plugin>
+    </gazebo>
 </robot>

Commit message: fortress BRANCH as classic is EOL

File: urdf/camera.xacro (robot description, xacro)
@@ -25,14 +25,3 @@
         <origin xyz="${0.5*(main_base_length+camera_length)} 0 0" rpy="0 0 0" />
     </joint>
-    <gazebo reference="camera" >
-        <material>Gazebo/Black</material>
-        <sensor name="camera_sensor" type="camera">
-            <pose>0 0 0 0 0 0</pose>
-            <visualize>true</visualize>
-            <update_rate>10.0</update_rate>
-            <plugin name="camera_controller" filename="libgazebo_ros_camera.so">
-                <frame_name>camera</frame_name>
-            </plugin>
-        </sensor>
-    </gazebo>
 </robot>

File: urdf/robot_arm.xacro (robot description, xacro)
@@ -81,15 +81,3 @@
         <limit effort="100" velocity="100" lower="0" upper="${pi/2}" />
     </joint>
-    <gazebo>
-        <plugin name="joint_state_publisher_controller" filename="libgazebo_ros_joint_state_publisher.so">
-            <update_rate>10</update_rate>
-            <joint_name>forearm_to_base</joint_name>
-            <joint_name>hand_to_forearm</joint_name>
-        </plugin>
-    </gazebo>
-    <gazebo>
-        <plugin name="joint_pose_trajectory_controller" filename="libgazebo_ros_joint_pose_trajectory.so">
-            <update_rate>2</update_rate>
-        </plugin>
-    </gazebo>
 </robot>

File: urdf/robot_gazebo.xacro (robot description, xacro)
@@ -24,25 +24,3 @@
         <mu2 value="0.1" />
     </gazebo>
-    <gazebo>
-        <plugin name="gazebo_ros_diff_drive" filename="libgazebo_ros_diff_drive.so">
-            <!-- Update rate in Hz -->
-            <update_rate>50</update_rate>
-            <!-- wheels -->
-            <left_joint>base_left_wheel_joint</left_joint>
-            <right_joint>base_right_wheel_joint</right_joint>
-            <max_wheel_torque>20</max_wheel_torque>
-            <max_wheel_acceleration>2.0</max_wheel_acceleration>
-            <command_topic>cmd_vel</command_topic>
-            <!-- kinematics -->
-            <wheel_separation>${main_base_width + wheel_length}</wheel_separation>
-            <wheel_diameter>${2*wheel_radius}</wheel_diameter>
-            <!-- output -->
-            <publish_odom>true</publish_odom>
-            <publish_odom_tf>true</publish_odom_tf>
-            <publish_wheel_tf>true</publish_wheel_tf>
-            <odometry_topic>odom</odometry_topic>
-            <odometry_frame>odom</odometry_frame>
-            <robot_base_frame>base_footprint</robot_base_frame>
-        </plugin>
-    </gazebo>
 </robot>
